File: pwm_radar/pwm_radar.kicad_pcb (KiCad board)
At the start: 2 copper layers, 39 x 39 mm, 22 parts, among them J1 Conn_Coaxial, J2 Conn_01x01_Pin, J3 Conn_01x01_Pin, J4 Conn_Coaxial, J5 Conn_Coaxial, J6 Conn_Coaxial, J7 Conn_01x01_Pin, J8 Conn_01x01_Pin

Commit message: added ant
added antenna
Parts:
- moved C6 2.54 mm to (109.9, 61.5), turned to 0 degrees
- moved C1 2.41 mm to (110.3, 54.2), turned to 0 degrees
Routing:
- net VDD: track 6.58 -> 5.77 mm
