File: pwm_radar/pwm_radar.kicad_pcb (KiCad board)
At the start: 2 copper layers, 39 x 39 mm, 22 parts, among them J1 Conn_Coaxial, J2 Conn_01x01_Pin, J3 Conn_01x01_Pin, J4 Conn_Coaxial, J5 Conn_Coaxial, J6 Conn_Coaxial, J7 Conn_01x01_Pin, J8 Conn_01x01_Pin

Commit message: added vivaldi antenna
added vivaldi antenna
Parts:
- removed H1, H2, H3, H4: MountingHole_Pad, MountingHole:MountingHole_2.5mm_Pad_Via
- added C1: 10u, Capacitor_SMD:C_0402_1005Metric_Pad0.74x0.62mm_HandSolder, B.Cu at (197.0, 64.9)
- added C2: 100p, Capacitor_SMD:C_0402_1005Metric_Pad0.74x0.62mm_HandSolder, B.Cu at (194.7, 65.3)
- added C3: 100p, Capacitor_SMD:C_0402_1005Metric_Pad0.74x0.62mm_HandSolder, B.Cu at (194.7, 66.4)
- added C4: 10u, Capacitor_SMD:C_0402_1005Metric_Pad0.74x0.62mm_HandSolder, B.Cu at (194.1, 70.8)
- added C5: 100n, Capacitor_SMD:C_0402_1005Metric_Pad0.74x0.62mm_HandSolder, B.Cu at (194.2, 71.9)
- added C6: 100p, Capacitor_SMD:C_0402_1005Metric_Pad0.74x0.62mm_HandSolder, B.Cu at (196.6, 72.3)
- added J1: Conn_Coaxial, pwm_radar_lib:Wurth_RF_PWM_Conn, F.Cu at (170.3, 67.8)
- added J2: Conn_01x01_Pin, Connector_PinHeader_1.00mm:PinHeader_1x01_P1.00mm_Vertical, B.Cu at (191.6, 67.4)
- added J3: Conn_01x01_Pin, Connector_PinHeader_1.00mm:PinHeader_1x01_P1.00mm_Vertical, B.Cu at (196.6, 66.4)
- added J4: Conn_Coaxial, pwm_radar_lib:Wurth_RF_PWM_Conn, F.Cu at (216.7, 86.8)
- added J5: Conn_Coaxial, pwm_radar_lib:Wurth_RF_PWM_Conn, F.Cu at (169.7, 86.8)
- added J7: Conn_01x01_Pin, Connector_PinHeader_1.00mm:PinHeader_1x01_P1.00mm_Vertical, B.Cu at (194.1, 69.1)
- added J8: Conn_01x01_Pin, Connector_PinHeader_1.00mm:PinHeader_1x01_P1.00mm_Vertical, B.Cu at (196.5, 70.8)
- added R1: 0, Resistor_SMD:R_0402_1005Metric_Pad0.72x0.64mm_HandSolder, F.Cu at (194.1, 67.4)
- added R2: 0, Resistor_SMD:R_0402_1005Metric_Pad0.72x0.64mm_HandSolder, F.Cu at (196.8, 68.5)
- added U1: ~, pwm_radar_lib:MC1630-1_MNC, F.Cu at (184.7, 67.8)
- added U2: ~, pwm_radar_lib:ADRF5020BCCZN, F.Cu at (200.7, 67.8)
- added U5: ~, RF_Antenna:Vivaldi Antenna 10 to 24 GHz, B.Cu at (197.7, 52.9)
Connections:
- U2 pad 21: GND -> (no net)
Routing:
- net Net-(J4-In): track 38.0 -> 76.0 mm
- net RF1+: track 19.8 -> 39.6 mm
- net RF1-: track 19.8 -> 39.6 mm
- net Net-(J6-In): track 8.81 -> 22.2 mm
- net VSS: track 8.63 -> 17.3 mm
- net VDD: track 5.77 -> 13.7 mm
- net Net-(J1-In): track 7.95 -> 15.9 mm
- net GND: track 6.12 -> 12.2 mm, vias 416 -> 832
- net CTRL: track 4.75 -> 9.50 mm
- net Net-(J7-Pin_1): track 2.39 -> 4.78 mm
- net EN: track 2.13 -> 4.25 mm
- net Net-(J2-Pin_1): track 1.92 -> 3.85 mm
Other:
- board size 39 x 39 mm -> 149.8 x 49.8 mm

Commit message: Update pwm_radar.kicad_pcb
Routing:
- net GND: vias 832 -> 522

Commit message: fixing some final touches
Parts:
- removed the J4 at (216.7, 86.8)
- removed the J5 at (169.7, 86.8)
Connections:
- U2 pad 3: Net-(J6-In) -> Net-(U4-RFC)
Routing:
- net Net-(J4-In): track 76.0 -> 38.0 mm
- net Net-(J6-In): track 22.2 -> 8.58 mm
- net Net-(U4-RFC): track 0.00 -> 13.2 mm
- net RF1-: track 39.6 -> 39.0 mm
- net GND: vias 522 -> 379
Other:
- board size 149.8 x 49.8 mm -> 149.8 x 39 mm

Commit message: fixed some issues
fixed issues
Connections:
- U2 pad 21: (no net) -> GND
Routing:
- net GND: vias 379 -> 413
- net (no net): vias 0 -> 1
Other:
- outline, holes or cut-outs redrawn

Commit message: final_checking
final_checking
Parts:
- removed the C1 at (197.0, 64.9)
- removed the C2 at (194.7, 65.3)
- removed the C3 at (194.7, 66.4)
- removed the C4 at (194.1, 70.8)
- removed the C5 at (194.2, 71.9)
- removed the C6 at (196.6, 72.3)
- removed the J1 at (170.3, 67.8)
- removed the J2 at (191.6, 67.4)
- removed the J3 at (196.6, 66.4)
- removed J4: Conn_Coaxial, pwm_radar_lib:Wurth_RF_PWM_Conn
- removed the J7 at (194.1, 69.1)
- removed the J8 at (196.5, 70.8)
- removed the R1 at (194.1, 67.4)
- removed the R2 at (196.8, 68.5)
- removed the U1 at (184.7, 67.8)
- removed the U2 at (200.7, 67.8)
- removed U5: ~, RF_Antenna:Vivaldi Antenna 10 to 24 GHz
- added J5: Conn_Coaxial, pwm_radar_lib:Wurth_RF_PWM_Conn, F.Cu at (116.9, 76.0)
Routing:
- net RF1+: track 39.1 -> 19.5 mm
- net RF1-: track 39.0 -> 19.5 mm
- net Net-(U4-RFC): track 13.2 -> 0.00 mm
- net VSS: track 17.3 -> 8.63 mm
- net Net-(J1-In): track 15.9 -> 7.95 mm
- net VDD: track 13.7 -> 6.82 mm
- net GND: track 12.2 -> 6.12 mm, vias 413 -> 280
- net CTRL: track 9.50 -> 4.90 mm
- net Net-(J7-Pin_1): track 4.78 -> 2.39 mm
- net EN: track 4.25 -> 2.15 mm
- net Net-(J2-Pin_1): track 3.85 -> 1.92 mm
- net (no net): vias 1 -> 0
Other:
- board size 149.8 x 39 mm -> 39 x 39 mm

Commit message: gerbers
gerbers
Parts:
- removed the J5 at (116.9, 76.0)
- added J4: Conn_Coaxial, pwm_radar_lib:Wurth_RF_PWM_Conn, F.Cu at (117.0, 76.0)
- moved J5 13.0 mm to (96.0, 76.0), turned to -90 degrees
- moved J1 12.9 mm to (96.5, 57.0), turned to -90 degrees
Connections:
- U2 pad 21: GND -> (no net)

Commit message: final gerbs v1
final gerbs v1
Parts:
- moved C4 3.46 mm to (109.9, 57.6)
- moved C5 1.28 mm to (107.5, 59.9)
- moved C6 0.96 mm to (110.5, 60.8)
- moved J8 0.73 mm to (109.9, 59.3)
Connections:
- U2 pad 21: (no net) -> GND
Routing:
- net GND: track 6.12 -> 20.3 mm, vias 280 -> 320
- net Net-(J6-In): track 8.58 -> 13.6 mm
- net Net-(J1-In): track 7.95 -> 12.9 mm
- net Net-(J4-In): track 38.0 -> 42.7 mm
