File: pwm_radar/vivaldi_ant/vivaldi_ant.kicad_pcb (KiCad board)
At the start: 2 copper layers, 34.1 x 20 mm, 1 part, among them J6 Conn_Coaxial

Commit message: added vivaldi antenna
added vivaldi antenna
Parts:
- moved J6 13.0 mm to (131.5, 85.0), turned to -90 degrees
Changed lines of the file:
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@@
 	(footprint "pwm_radar_lib:Wurth_RF_PWM_Conn"
 		(layer "B.Cu")
-		(at 144.5 85 90)
+		(at 131.519471 85 -90)
 		(property "Reference" "J6"
-			(at -9.9 -4 270)
+			(at -9.9 -4 90)
 			(unlocked yes)
 			(layer "B.SilkS")
@@
 		)
 		(property "Value" "Conn_Coaxial"
-			(at 0 -1 270)
+			(at 0 -1 90)
 			(unlocked yes)
 			(layer "B.Fab")
@@
 		)
 		(property "Datasheet" ""
-			(at 0 0 270)
+			(at 0 0 90)
 			(unlocked yes)
 			(layer "B.Fab")
@@
 		)
 		(property "Description" "coaxial connector (BNC, SMA, SMB, SMC, Cinch/RCA, LEMO, ...)"
-			(at 0 0 270)
+			(at 0 0 90)
 			(unlocked yes)
 			(layer "B.Fab")
@@
 		)
 		(attr smd)
+		(fp_line
+			(start -0.2 -3.9)
+			(end 0.2 -3.9)
+			(stroke
+				(width 0.1)
+				(type default)
+			)
+			(layer "B.SilkS")
+		)
+		(fp_line
+			(start 7 -4)
+			(end 7 -9)
+			(stroke
+				(width 0.1)
+				(type default)
+			)
+			(layer "B.SilkS")
+		)
 		(fp_line
 			(start -7 -9)
@@
 			(layer "B.SilkS")
 		)
-		(fp_line
-			(start 7 -4)
-			(end 7 -9)
-			(stroke
-				(width 0.1)
-				(type default)
-			)
-			(layer "B.SilkS")
-		)
-		(fp_line
-			(start -0.2 -3.9)
-			(end 0.2 -3.9)
-			(stroke
-				(width 0.1)
-				(type default)
-			)
-			(layer "B.SilkS")
+		(fp_circle
+			(center -4.75 -6.5)
+			(end -4.75 -7.5)
+			(stroke
+				(width 0.1)
+				(type solid)
+			)
+			(fill yes)
+			(layer "Edge.Cuts")
 		)
 		(fp_circle
@@
 			(layer "Edge.Cuts")
 		)
-		(fp_circle
-			(center -4.75 -6.5)
-			(end -4.75 -7.5)
-			(stroke
-				(width 0.1)
-				(type solid)
-			)
-			(fill yes)
-			(layer "Edge.Cuts")
-		)
 		(fp_text user "${REFERENCE}"
-			(at 0 -2.5 270)
+			(at 0 -2.5 90)
 			(unlocked yes)
 			(layer "B.Fab")
@@
 		)
 		(pad "1" connect rect
-			(at 0 -6.5 90)
+			(at 0 -6.5 270)
 			(size 0.4 5.2)
 			(layers "B.Cu" "B.Mask")
@@
 		)
 		(pad "2" connect rect
-			(at -4.475 -6.5 90)
+			(at -4.475 -6.5 270)
 			(size 5.15 5.2)
 			(layers "B.Cu" "B.Mask")
@@
 		)
 		(pad "2" connect rect
-			(at 0.025 -6.5 90)
+			(at 0.025 -6.5 270)
 			(size 14.15 5.2)
 			(layers "F.Cu" "F.Mask")
@@
 		)
 		(pad "2" connect rect
-			(at 4.55 -6.5 90)
+			(at 4.55 -6.5 270)
 			(size 5.1 5.2)
 			(layers "B.Cu" "B.Mask")
@@
 	)
 	(gr_line
-		(start 150.4 86.400002)
-		(end 149.9 84.600001)
+		(start 149.9 87.3)
+		(end 149.9 83.700001)
+		(stroke
+			(width 3)
+			(type default)
+		)
+		(layer "B.Mask")
+	)
+	(gr_line
+		(start 151.7 87.3)
+		(end 149.899999 87.3)
 		(stroke
 			(width 3)
@@
 	)
 	(via
-		(at 139.6 82.2)
-		(size 0.6)
-		(drill 0.3)
+		(at 140 82.3)
+		(size 0.6)
+		(drill 0.3)

Commit message: fixing some final touches
Parts:
- added U1: ~, RF_Antenna:Vivaldi Antenna 10 to 24 GHz, F.Cu at (130.2, 95.0)
- moved J6 6.77 mm to (136.2, 80.1)
Routing:
- net Net-(AE1-PCB_Trace): track 12.6 -> 0.00 mm
- net GND: vias 8 -> 0
- removed copper zone on B.Cu, net Net-(AE1-PCB_Trace)
Other:
- board size 34.1 x 20 mm -> 29.3 x 21.7 mm

Commit message: fixed some issues
fixed issues
Changed lines of the file:
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@@
 			(layer "B.SilkS")
-		)
-		(fp_circle
-			(center -4.75 -6.5)
-			(end -4.75 -7.5)
-			(stroke
-				(width 0.1)
-				(type solid)
-			)
-			(fill yes)
-			(layer "Edge.Cuts")
-		)
-		(fp_circle
-			(center 4.75 -6.5)
-			(end 4.75 -7.5)
-			(stroke
-				(width 0.1)
-				(type solid)
-			)
-			(fill yes)
-			(layer "Edge.Cuts")
 		)
 		(fp_text user "${REFERENCE}"
@@
 			(thermal_bridge_angle 45)
 		)
-		(pad "2" connect rect
+		(pad "2" thru_hole rect
 			(at -4.475 -6.5 270)
 			(size 5.15 5.2)
-			(layers "B.Cu" "B.Mask")
+			(drill 2)
+			(layers "*.Cu" "*.Mask")
+			(remove_unused_layers no)
 			(net 1 "GND")
 			(pinfunction "Ext")
@@
 			(thermal_bridge_angle 45)
 		)
-		(pad "2" connect rect
+		(pad "2" thru_hole rect
 			(at 4.55 -6.5 270)
 			(size 5.1 5.2)
-			(layers "B.Cu" "B.Mask")
+			(drill 2)
+			(layers "*.Cu" "*.Mask")
+			(remove_unused_layers no)
 			(net 1 "GND")
 			(pinfunction "Ext")
@@
 		(layer "B.Cu")
 	)
+	(gr_line
+		(start 149.9 84.600001)
+		(end 149.9 82.8)
+		(stroke
+			(width 3)
+			(type default)
+		)
+		(layer "B.Mask")
+	)
 	(gr_rect
 		(start 139.77 77.47)
@@
 		(stroke
 			(width 3)
-			(type default)
-		)
-		(layer "B.Mask")
-	)
-	(gr_line
-		(start 149.9 84.600001)
-		(end 149.9 82.8)
-		(stroke
-			(width 3)

Commit message: final_checking
final_checking
Changed lines of the file:
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@@
 	(generator_version "9.0")
 	(general
-		(thickness 1.6)
+		(thickness 0.6)
 		(legacy_teardrops no)
 	)
@@
 	)
 	(setup
+		(stackup
+			(layer "F.SilkS"
+				(type "Top Silk Screen")
+			)
+			(layer "F.Paste"
+				(type "Top Solder Paste")
+			)
+			(layer "F.Mask"
+				(type "Top Solder Mask")
+				(thickness 0.01)
+			)
+			(layer "F.Cu"
+				(type "copper")
+				(thickness 0.035)
+			)
+			(layer "dielectric 1"
+				(type "core")
+				(thickness 0.51)
+				(material "Rogers RO4350B")
+				(epsilon_r 3.66)
+				(loss_tangent 0.00035)
+			)
+			(layer "B.Cu"
+				(type "copper")
+				(thickness 0.035)
+			)
+			(layer "B.Mask"
+				(type "Bottom Solder Mask")
+				(thickness 0.01)
+			)
+			(layer "B.Paste"
+				(type "Bottom Solder Paste")
+			)
+			(layer "B.SilkS"
+				(type "Bottom Silk Screen")
+			)
+			(copper_finish "None")
+			(dielectric_constraints no)
+		)
 		(pad_to_mask_clearance 0)
 		(allow_soldermask_bridges_in_footprints no)
@@
 			(outputformat 1)
 			(mirror no)
-			(drillshape 1)
+			(drillshape 0)
 			(scaleselection 1)
-			(outputdirectory "")
+			(outputdirectory "../Gerbers/ANT/")
 		)
 	)
@@
 	)
 	(gr_rect
-		(start 140.15 79.604997)
-		(end 145.15 80.604997)
+		(start 140.05 79.604997)
+		(end 148.85 80.604997)
 		(stroke
 			(width 0)
@@
 		(fill yes)
 		(layer "B.Cu")
-	)
-	(gr_line
-		(start 149.9 84.600001)
-		(end 149.9 82.8)
-		(stroke
-			(width 3)
-			(type default)
-		)
-		(layer "B.Mask")
 	)
 	(gr_rect
@@
 		(stroke
 			(width 3)
+			(type default)
+		)
+		(layer "B.Mask")
+	)
+	(gr_line
+		(start 149.9 84.600001)
+		(end 149.9 82.8)
+		(stroke
+			(width 3)

Commit message: gerbers
gerbers
Parts:
- moved J6 12.9 mm to (149.0, 80.1), turned to 90 degrees
Changed lines of the file:
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@@
 	(footprint "pwm_radar_lib:Wurth_RF_PWM_Conn"
 		(layer "B.Cu")
-		(at 136.15 80.065 -90)
+		(at 149 80.104997 90)
 		(property "Reference" "J6"
-			(at -9.9 -4 90)
+			(at -9.9 -4 270)
 			(unlocked yes)
 			(layer "B.SilkS")
@@
 		)
 		(property "Value" "Conn_Coaxial"
-			(at 0 -1 90)
+			(at 0 -1 270)
 			(unlocked yes)
 			(layer "B.Fab")
@@
 		)
 		(property "Datasheet" ""
-			(at 0 0 90)
+			(at 0 0 270)
 			(unlocked yes)
 			(layer "B.Fab")
@@
 		)
 		(property "Description" "coaxial connector (BNC, SMA, SMB, SMC, Cinch/RCA, LEMO, ...)"
-			(at 0 0 90)
+			(at 0 0 270)
 			(unlocked yes)
 			(layer "B.Fab")
@@
 		(attr smd)
 		(fp_line
-			(start -0.2 -3.9)
-			(end 0.2 -3.9)
+			(start -7 -9)
+			(end -7 -4)
 			(stroke
 				(width 0.1)
@@
 			(layer "B.SilkS")
 		)
-		(fp_line
-			(start -7 -9)
-			(end -7 -4)
-			(stroke
-				(width 0.1)
-				(type default)
-			)
-			(layer "B.SilkS")
-		)
 		(fp_text user "${REFERENCE}"
-			(at 0 -2.5 90)
+			(at 0 -2.5 270)
 			(unlocked yes)
 			(layer "B.Fab")
@@
 		)
 		(pad "1" connect rect
-			(at 0 -6.5 270)
+			(at 0 -6.5 90)
 			(size 0.4 5.2)
 			(layers "B.Cu" "B.Mask")
@@
 		)
 		(pad "2" thru_hole rect
-			(at -4.475 -6.5 270)
-			(size 5.15 5.2)
-			(drill 2)
+			(at -4.7 -6.2 90)
+			(size 6 5)
+			(drill 2.5
+				(offset 0.675 -0.3)
+			)
 			(layers "*.Cu" "*.Mask")
 			(remove_unused_layers no)
@@
 		)
 		(pad "2" connect rect
-			(at 0.025 -6.5 270)
-			(size 14.15 5.2)
+			(at 0.025 -6.5 90)
+			(size 14 5)
 			(layers "F.Cu" "F.Mask")
 			(net 1 "GND")
@@
 		)
 		(pad "2" thru_hole rect
-			(at 4.55 -6.5 270)
-			(size 5.1 5.2)
-			(drill 2)
+			(at 4.7 -6.2 270)
+			(size 6 5)
+			(drill 2.5
+				(offset 0.675 0.3)
+			)
 			(layers "*.Cu" "*.Mask")
 			(remove_unused_layers no)
@@
 		)
 		(embedded_fonts no)
+		(model "C:/Users/flatr/Downloads/STP_ConSMA_60312862112552_rev1.stp"
+			(offset
+				(xyz 0 -11.2 0)
+			)
+			(scale
+				(xyz 1 1 1)
+			)
+			(rotate
+				(xyz -0 -0 -180)
+			)
+		)
 	)
 	(gr_rect
@@
 		(fill yes)
 		(layer "B.Cu")
+		(net 3)
+	)
+	(gr_line
+		(start 149.9 84.600001)
+		(end 149.9 82.8)
+		(stroke
+			(width 3)
+			(type default)
+		)
+		(layer "B.Mask")
 	)
 	(gr_rect
@@
 		(stroke
 			(width 3)
-			(type default)
-		)
-		(layer "B.Mask")
-	)
-	(gr_line
-		(start 149.9 84.600001)
-		(end 149.9 82.8)
-		(stroke
-			(width 3)

Commit message: final gerbs v1
final gerbs v1
Routing:
- net Net-(J4-In): track 0.00 -> 5.00 mm
Other:
- board size 29.3 x 21.7 mm -> 29.3 x 23.3 mm
Changed lines of the file:
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@@
 	(net 2 "Net-(AE1-PCB_Trace)")
 	(net 3 "Net-(J1-Ext)")
+	(net 4 "Net-(J4-In)")
 	(footprint "RF_Antenna:Vivaldi Antenna 10 to 24 GHz"
 		(layer "F.Cu")
@@
 	)
 	(gr_rect
+		(start 143.83 93.92)
+		(end 168.94 96.01)
+		(stroke
+			(width 0.2)
+			(type solid)
+		)
+		(fill yes)
+		(layer "F.Cu")
+		(net 1)
+	)
+	(gr_rect
 		(start 133.6 71.9)
 		(end 172.4 100.6)
@@
 		(net 3)
 	)
-	(gr_line
-		(start 149.9 84.600001)
-		(end 149.9 82.8)
-		(stroke
-			(width 3)
-			(type default)
-		)
-		(layer "B.Mask")
-	)
 	(gr_rect
 		(start 139.77 77.47)
@@
 		(layer "B.Mask")
 	)
-	(gr_rect
-		(start 140.02 73.03)
+	(gr_line
+		(start 149.9 84.600001)
+		(end 149.9 82.8)
+		(stroke
+			(width 3)
+			(type default)
+		)
+		(layer "B.Mask")
+	)
+	(gr_line
+		(start 140.02 94.76)
+		(end 140.02 73.03)
+		(stroke
+			(width 0.05)
+			(type default)
+		)
+		(layer "Edge.Cuts")
+	)
+	(gr_line
+		(start 140.02 96.37)
+		(end 140.02 94.76)
+		(stroke
+			(width 0.05)
+			(type default)
+		)
+		(layer "Edge.Cuts")
+	)
+	(gr_line
+		(start 169.29 73.03)
+		(end 140.02 73.03)
+		(stroke
+			(width 0.05)
+			(type default)
+		)
+		(layer "Edge.Cuts")
+	)
+	(gr_line
+		(start 169.29 73.03)
 		(end 169.29 94.76)
 		(stroke
@@
 			(type default)
 		)
-		(fill no)
-		(layer "Edge.Cuts")
+		(layer "Edge.Cuts")
+	)
+	(gr_line
+		(start 169.29 94.76)
+		(end 169.29 96.36)
+		(stroke
+			(width 0.05)
+			(type default)
+		)
+		(layer "Edge.Cuts")
+	)
+	(gr_line
+		(start 169.29 96.36)
+		(end 140.02 96.369993)
+		(stroke
+			(width 0.05)
+			(type default)
+		)
+		(layer "Edge.Cuts")
+	)
+	(segment
+		(start 143.55 80.1)
+		(end 140.25 80.1)
+		(width 1.1)
+		(layer "B.Cu")
+		(net 4)
+	)
+	(segment
+		(start 143.55 80.1)
+		(end 145.25 80.1)
+		(width 1.1)
+		(layer "B.Cu")
+		(net 4)
 	)
 	(zone
