File: pwm_radar/pwm_radar_with_antenna/pwm_radar_with_antenna.kicad_pcb (KiCad board)
At the start: 2 copper layers, 62.6 x 29.3 mm, 16 parts, among them J1 Conn_Coaxial, J2 Conn_01x01_Pin, J3 Conn_01x01_Pin, J7 Conn_01x01_Pin, J8 Conn_01x01_Pin

Commit message: gerbers
gerbers
Parts:
- moved J1 12.9 mm to (117.0, 89.5), turned to -90 degrees

Commit message: final gerbs v1
final gerbs v1
Parts:
- added H1: MountingHole_Pad, MountingHole:MountingHole_3.2mm_M3_DIN965_Pad_TopBottom, F.Cu at (111.6, 78.3)
- added H2: MountingHole_Pad, MountingHole:MountingHole_3.2mm_M3_DIN965_Pad_TopBottom, F.Cu at (111.6, 100.5)
- added H3: MountingHole_Pad, MountingHole:MountingHole_3.2mm_M3_DIN965_Pad_TopBottom, F.Cu at (142.2, 100.4)
- added H4: MountingHole_Pad, MountingHole:MountingHole_3.2mm_M3_DIN965_Pad_TopBottom, F.Cu at (142.2, 78.1)
- moved C6 3.73 mm to (130.4, 90.2)
- moved C4 2.23 mm to (130.0, 93.3)
- moved C5 1.29 mm to (128.0, 92.3)
- moved J8 0.63 mm to (130.3, 91.8)
Routing:
- net GND: track 6.12 -> 20.5 mm, vias 135 -> 223
- net Net-(J1-In): track 7.95 -> 12.9 mm
Other:
- outline, holes or cut-outs redrawn
- board text added: "PWM Radar V1 CNDE AMNTL"
- board text added: "fdreshaj 26"
