File: pwm_radar/pwm_radar_with_antenna/pwm_radar_with_antenna.kicad_sch (KiCad schematic)
At the start: 18 parts, among them J1 Conn_Coaxial, J2 Conn_01x01_Pin, J3 Conn_01x01_Pin, J4 Conn_Coaxial, J5 Conn_Coaxial, J6 Conn_Coaxial, J7 Conn_01x01_Pin, J8 Conn_01x01_Pin

Commit message: final_checking
final_checking
Parts:
- removed C1, C4: 10u, Capacitor_SMD:C_0402_1005Metric_Pad0.74x0.62mm_HandSolder, symbol Device:C
- removed C2, C3, C6: 100p, Capacitor_SMD:C_0402_1005Metric_Pad0.74x0.62mm_HandSolder, symbol Device:C
- removed C5: 100n, Capacitor_SMD:C_0402_1005Metric_Pad0.74x0.62mm_HandSolder, symbol Device:C
- removed J1, J4, J5, J6: Conn_Coaxial, pwm_radar_lib:Wurth_RF_PWM_Conn, symbol Connector:Conn_Coaxial
- removed J2, J3, J7, J8: Conn_01x01_Pin, Connector_PinHeader_1.00mm:PinHeader_1x01_P1.00mm_Vertical, symbol Connector:Conn_01x01_Pin
- removed R1, R2: 0, Resistor_SMD:R_0402_1005Metric_Pad0.72x0.64mm_HandSolder, symbol Device:R
- removed U1: ~, pwm_radar_lib:MC1630-1_MNC, symbol pwm_radar_library:MTY-243+
- removed U2: ~, pwm_radar_lib:ADRF5020BCCZN, symbol pwm_radar_library:ADRF5020
- added C10, C7: 10u, Capacitor_SMD:C_0402_1005Metric_Pad0.74x0.62mm_HandSolder, symbol Device:C
- added C11: 100n, Capacitor_SMD:C_0402_1005Metric_Pad0.74x0.62mm_HandSolder, symbol Device:C
- added C12, C8, C9: 100p, Capacitor_SMD:C_0402_1005Metric_Pad0.74x0.62mm_HandSolder, symbol Device:C
- added J10, J11, J12, J13: Conn_01x01_Pin, Connector_PinHeader_1.00mm:PinHeader_1x01_P1.00mm_Vertical, symbol Connector:Conn_01x01_Pin
- added J9: Conn_Coaxial, pwm_radar_lib:Wurth_RF_PWM_Conn, symbol Connector:Conn_Coaxial
- added R3, R4: 0, Resistor_SMD:R_0402_1005Metric_Pad0.72x0.64mm_HandSolder, symbol Device:R
- added U3: ~, pwm_radar_lib:MC1630-1_MNC, symbol pwm_radar_library:MTY-243+
- added U4: ~, pwm_radar_lib:ADRF5020BCCZN, symbol pwm_radar_library:ADRF5020
- added U5: ~, symbol antenna_lib:Vivaldi_Antenna_10_24
Connections:
- net CTRL: now also R3.1, U4.12 (CTRL)
- net EN: now also R4.1, U4.14 (EN)
- net GND: now also C10.2, C11.2, C12.2, C7.2, C8.2, C9.2, J9.2 (Ext), U3.1 (GND), U3.3 (GND), U3.5 (NC), U3.7 (GND_PAD), U4.1 (GND), U4.10 (GND), U4.13 (GND), U4.16 (GND), U4.17 (GND), U4.19 (GND), U4.2 (GND), U4.20 (GND), U4.4 (GND), U4.5 (GND), U4.6 (GND), U4.7 (GND), U4.9 (GND), U5. (Gnd)
- net RF1+: now also U3.6 (Secondary_Dot), U4.8 (RF1)
- net RF1-: now also U3.4 (Secondary)
- net VDD: now also C7.1, C8.1, C9.1, J10.1 (Pin_1), U4.11 (VDD)
- net VSS: now also C10.1, C11.1, C12.1, J12.1 (Pin_1), U4.15 (VSS)
- new net: J9.1 (In), U3.2 (Primary)
- new net: J11.1 (Pin_1), R4.2
- new net: U4.3 (RFC), U5.1 (Ant_In)
- new net: J13.1 (Pin_1), R3.2
Other:
- note removed: "THRU Cal"
- company: Center for Non Destructive Evaluation -> (none)
- title: PWM Phased Array Radar -> (none)

Commit message: final gerbs v1
final gerbs v1
Parts:
- added H1, H2, H3, H4: MountingHole_Pad, MountingHole:MountingHole_3.2mm_M3_DIN965_Pad_TopBottom, symbol Mechanical:MountingHole_Pad
Connections:
- net GND: now also H1.1, H2.1, H3.1, H4.1
